File: exploere202.kicad_pcb (KiCad board)
At the start: 2 copper layers, 47 x 80 mm, 60 parts, among them J1 External power supply 12V/18V, J2 9V Battery, J4 Conn_Coaxial, J5 AudioJack3, J6 AudioJack3, Q1 BC237, Q2 BC237, SW1 PWR, SW2 HPF, T1 Transformer_Audio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

Commit message: Add files via upload
Parts:
- removed the G*** at (151.0, 96.5)
- removed the G*** at (163.8, 92.9)
- added G***: LOGO, LOGO, F.Cu at (146.2, 60.0)
- added G***: LOGO, LOGO, F.Cu at (157.0, 130.9)
- added G***: LOGO, LOGO, F.Cu at (165.8, 96.8)
- moved C10 1.10 mm to (168.0, 119.2)
Routing:
- net Net-(U2--): track 18.8 -> 19.9 mm
- net Net-(D2-K): track 38.5 -> 39.5 mm

Commit message: Add files via upload
Parts:
- moved C1 1.38 mm to (144.2, 95.7)
- moved SW2 1.38 mm to (138.5, 96.9)
Routing:
- net 1/2: track 41.3 -> 42.6 mm
- net Net-(T1-SA): track 17.8 -> 18.6 mm
Other:
- outline, holes or cut-outs redrawn

Commit message: Add files via upload
Parts:
- removed the G*** at (157.0, 130.9)
- removed the REF** at (179.0, 56.5)
- removed the REF** at (137.0, 56.5)
- removed the REF** at (137.0, 131.5)
- removed the REF** at (179.0, 131.5)
- added H1: MountingHole_Pad, MountingHole:MountingHole_2.1mm, F.Cu at (179.0, 55.1)
- added H2: MountingHole_Pad, MountingHole:MountingHole_2.1mm, F.Cu at (137.0, 55.1)
- added H3: MountingHole_Pad, MountingHole:MountingHole_2.1mm, F.Cu at (137.0, 131.5)
- added H4: MountingHole_Pad, MountingHole:MountingHole_2.1mm, F.Cu at (179.0, 131.5)
- moved G*** 6.41 mm to (139.9, 59.0)
- moved TP4 2.75 mm to (142.6, 83.3)
- moved J1 2.52 mm to (136.3, 78.9), turned to 90 degrees
- moved D1 2.20 mm to (141.6, 78.2)
- moved D3 2.10 mm to (137.9, 82.2)
- moved R1 2.10 mm to (139.2, 81.7)
Routing:
- net Net-(D1-A): track 2.62 -> 0.00 mm
- net Net-(T1-SA): track 18.6 -> 17.4 mm
- net VCC: track 33.1 -> 32.3 mm
- net GND: vias 14 -> 39
Other:
- board size 47 x 80 mm -> 47 x 81.5 mm
- board text added: "By ambraglow v0.1"
- board text added: "meow :3"

Commit message: Add files via upload
Parts:
- added G***: LOGO, LOGO, F.Cu at (170.9, 128.5)
- moved NE1 10.2 mm to (171.8, 74.4), turned to 180 degrees
- moved TP1 9.01 mm to (155.5, 80.8)
- moved TP2 6.71 mm to (148.7, 114.9)
- moved C5 1.61 mm to (164.2, 86.0)
- moved R7 1.61 mm to (166.7, 85.2)
- moved R5 1.61 mm to (164.2, 84.5)
- moved TP5 1.49 mm to (167.4, 116.4)
- moved G*** 1.19 mm to (139.2, 58.0)
- moved C10 0.70 mm to (168.2, 119.8)
- moved C11 0.40 mm to (152.2, 101.6)
- moved R10 0.40 mm to (149.0, 102.6)
- moved C8 0.32 mm to (157.7, 100.4)
- moved J1 0.20 mm to (136.1, 78.9)
Routing:
- net 1/2: track 42.6 -> 48.6 mm, vias 1 -> 2
- net Net-(C15-Pad2): track 12.7 -> 8.28 mm
- net Net-(D1-A): track 0.00 -> 2.97 mm
- net Net-(Q1-B): track 18.3 -> 21.2 mm
- net Net-(D2-K): track 39.7 -> 37.9 mm
- net Net-(C6-Pad2): track 4.56 -> 3.25 mm
- net Net-(Q1-C): track 16.6 -> 17.6 mm
- net Net-(C7-Pad2): track 29.4 -> 30.0 mm
- net GND: vias 39 -> 41
Other:
- board text added: "By ambraglow"
- board text added: "EXPLORER E202 DESIGN"
- board text added: "Laura said meow :3"
- board text added: "Phone_Out"
- board text removed: "By ambraglow v0.1"
- board text removed: "meow :3"

Commit message: Add files via upload
Parts:
- removed the G*** at (165.8, 96.8)
- C11, C2: footprint Capacitor_SMD:C_0603_1608Metric -> Capacitor_SMD:C_0805_2012Metric
- C12, C7, C9: footprint Capacitor_SMD:CP_Elec_4x5.4 -> Capacitor_SMD:CP_Elec_6.3x4.5
- C15: footprint Capacitor_SMD:CP_Elec_4x5.4 -> Capacitor_THT:CP_Radial_D6.3mm_P2.50mm
- D1, D2: footprint Diode_SMD:D_0603_1608Metric -> Diode_SMD:D_SOD-123
- TP1, TP2, TP4, TP5: footprint TestPoint:TestPoint_Pad_D1.5mm -> TestPoint:TestPoint_Pad_D2.5mm
- moved TP5 7.74 mm to (170.8, 123.3)
- moved D2 6.11 mm to (156.7, 65.7), turned to 90 degrees
- moved C9 5.31 mm to (166.3, 108.8)
- moved C13 4.55 mm to (154.7, 110.8), turned to 0 degrees
- moved TP2 4.26 mm to (149.1, 110.7)
- moved C12 3.16 mm to (159.4, 115.5), turned to -90 degrees
- moved D1 3.05 mm to (139.7, 75.8), turned to 180 degrees
- moved C15 2.99 mm to (152.1, 113.9)
- moved R9 2.72 mm to (162.8, 102.5), turned to -90 degrees
- moved T1 2.66 mm to (156.7, 125.4)
- moved TP3 2.21 mm to (150.1, 120.0)
- moved C10 2.17 mm to (169.4, 118.1)
- moved R12 2.00 mm to (151.7, 108.0), turned to -90 degrees
- moved C1 1.67 mm to (143.2, 94.3)
- moved C7 1.46 mm to (159.7, 97.2)
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Routing:
- net LINE OUT: track 8.56 -> 19.4 mm
- net Net-(C9-Pad1): track 12.5 -> 4.96 mm
- net Net-(C12-Pad2): track 4.10 -> 11.5 mm
- net B+: track 2.62 -> 6.76 mm
- net Net-(U2-BYPASS): track 7.82 -> 4.26 mm
- net Net-(C15-Pad2): track 8.28 -> 11.5 mm
- net Net-(U2--): track 20.0 -> 23.0 mm
- net Net-(C15-Pad1): track 2.72 -> 5.26 mm
- net Net-(T1-SA): track 17.4 -> 15.3 mm
- net Net-(C7-Pad2): track 30.0 -> 32.0 mm
- net Net-(T1-SB): track 11.0 -> 9.09 mm
- net Net-(R11-Pad1): track 4.61 -> 6.37 mm
- net Net-(Q1-C): track 17.6 -> 19.3 mm
- net 1/2: track 48.6 -> 49.9 mm
- net Net-(D2-K): track 37.9 -> 39.1 mm
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Other:
- board text added: "TODO: DONE - C12, C7, C9 and C15 - change package to THT or more common SMD one DONE - C11, C2 - change package 0603 -> 0805 DONE, changed footprint to SOD-123 - D1, D2 - find where to source DONE - find L1 on LCSC"
