File: exploere202.kicad_sch (KiCad schematic)
At the start: 52 parts, among them J1 External power supply 12V/18V, J2 9V Battery, J4 Conn_Coaxial, J5 AudioJack3, J6 AudioJack3, Q1 BC237, Q2 BC237, SW1 PWR, SW2 HPF, T1 Transformer_Audio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

Commit message: Add files via upload
Parts:
- added H1: MountingHole_Pad, MountingHole:MountingHole_2.1mm, symbol Mechanical:MountingHole_Pad
- added H2, H3, H4: MountingHole_Pad, project:MountingHole_2.1mm, symbol Mechanical:MountingHole_Pad
Connections:
- net GND: now also H1.1, H2.1, H3.1, H4.1

Commit message: Add files via upload
Parts:
- C11, C2: footprint Capacitor_SMD:C_0603_1608Metric -> Capacitor_SMD:C_0805_2012Metric
- C12, C7, C9: footprint Capacitor_SMD:CP_Elec_4x5.4 -> Capacitor_SMD:CP_Elec_6.3x4.5
- C15: footprint Capacitor_SMD:CP_Elec_4x5.4 -> Capacitor_THT:CP_Radial_D6.3mm_P2.50mm
- D1, D2: footprint Diode_SMD:D_0603_1608Metric -> Diode_SMD:D_SOD-123
- H2, H3, H4: footprint project:MountingHole_2.1mm -> MountingHole:MountingHole_2.1mm
- TP1, TP2, TP4, TP5: footprint TestPoint:TestPoint_Pad_D1.5mm -> TestPoint:TestPoint_Pad_D2.5mm
Changed lines of the file:
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@@
 			)
 		)
-		(property "Footprint" "Capacitor_SMD:CP_Elec_4x5.4"
+		(property "Footprint" "Capacitor_SMD:CP_Elec_6.3x4.5"
 			(at 198.12 135.89 0)
 			(effects
@@
 			)
 		)
-		(property "Footprint" "Diode_SMD:D_0603_1608Metric"
+		(property "Footprint" "Diode_SMD:D_SOD-123"
 			(at 58.42 55.88 0)
 			(effects
@@
 			)
 		)
-		(property "Footprint" "Capacitor_SMD:CP_Elec_4x5.4"
+		(property "Footprint" "Capacitor_THT:CP_Radial_D6.3mm_P2.50mm"
 			(at 227.33 121.92 0)
 			(effects
@@
 			)
 		)
-		(property "Footprint" "TestPoint:TestPoint_Pad_D1.5mm"
+		(property "Footprint" "TestPoint:TestPoint_Pad_D2.5mm"
 			(at 87.63 38.1 0)
 			(effects
@@
 			)
 		)
-		(property "Footprint" "Capacitor_SMD:C_0603_1608Metric"
+		(property "Footprint" "Capacitor_SMD:C_0805_2012Metric"
 			(at 124.46 102.87 0)
 			(effects
@@
 			)
 		)
-		(property "Footprint" "Capacitor_SMD:C_0603_1608Metric"
+		(property "Footprint" "Capacitor_SMD:C_0805_2012Metric"
 			(at 201.93 104.14 0)
 			(effects
@@
 			)
 		)
-		(property "Footprint" "Capacitor_SMD:CP_Elec_4x5.4"
+		(property "Footprint" "Capacitor_SMD:CP_Elec_6.3x4.5"
 			(at 149.86 119.6848 0)
 			(effects
@@
 			)
 		)
-		(property "Footprint" "project:MountingHole_2.1mm"
+		(property "Footprint" "MountingHole:MountingHole_2.1mm"
 			(at 195.58 30.48 0)
 			(effects
@@
 			)
 		)
-		(property "Footprint" "TestPoint:TestPoint_Pad_D1.5mm"
+		(property "Footprint" "TestPoint:TestPoint_Pad_D2.5mm"
 			(at 228.6 121.92 0)
 			(effects
@@
 			)
 		)
-		(property "Footprint" "TestPoint:TestPoint_Pad_D1.5mm"
+		(property "Footprint" "TestPoint:TestPoint_Pad_D2.5mm"
 			(at 152.4 95.25 0)
 			(effects
@@
 			)
 		)
-		(property "Footprint" "Capacitor_SMD:CP_Elec_4x5.4"
+		(property "Footprint" "Capacitor_SMD:CP_Elec_6.3x4.5"
 			(at 151.4348 101.6 0)
 			(effects
@@
 			)
 		)
-		(property "Footprint" "project:MountingHole_2.1mm"
+		(property "Footprint" "MountingHole:MountingHole_2.1mm"
 			(at 185.42 30.48 0)
 			(effects
@@
 			)
 		)
-		(property "Footprint" "TestPoint:TestPoint_Pad_D1.5mm"
+		(property "Footprint" "TestPoint:TestPoint_Pad_D2.5mm"
 			(at 115.57 55.88 0)
 			(effects
@@
 			)
 		)
-		(property "Footprint" "project:MountingHole_2.1mm"
+		(property "Footprint" "MountingHole:MountingHole_2.1mm"
 			(at 195.58 40.64 0)
 			(effects
@@
 			)
 		)
-		(property "Footprint" "Diode_SMD:D_0603_1608Metric"
+		(property "Footprint" "Diode_SMD:D_SOD-123"
 			(at 71.12 38.1 0)
 			(effects
